File: pcbs/tv-timer-pcbs/tv-timer-pcbs.kicad_pcb (KiCad board)
At the start: 2 copper layers, 30.4 x 51.7 mm, 9 parts, among them J1 Conn_01x03, J2 Conn_01x03

Commit message: Digit ready to go
Parts:
- D1, D2, D3, D4, D5, D6, D7: footprint ProjectLibrary:WS2812b_5mm_THT -> LED_THT:LED_D5.0mm-4_RGB_Wide_Pins
- moved D6 3.76 mm to (94.3, 61.4), turned to -90 degrees
- moved D7 1.36 mm to (108.8, 75.9)
- moved D4 1.34 mm to (102.3, 98.2)
- moved D1 1.32 mm to (108.7, 53.5)
- moved D3 1.32 mm to (116.7, 90.3)
- moved D2 1.31 mm to (116.7, 67.9)
- moved D5 1.28 mm to (94.3, 83.8)
Routing:
- net Net-(D5-DOUT): track 24.2 -> 18.9 mm
- net Net-(D6-DOUT): track 14.2 -> 17.9 mm
- net Net-(D1-DIN): track 30.1 -> 27.9 mm
- net Net-(D4-DOUT): track 13.1 -> 11.2 mm
- net Net-(D3-DOUT): track 13.1 -> 11.2 mm
- net Net-(D1-DOUT): track 13.1 -> 11.3 mm
- net Net-(D2-DOUT): track 20.3 -> 18.7 mm
- net Net-(D7-DOUT): track 9.74 -> 8.38 mm
Other:
- outline, holes or cut-outs redrawn
- board text added: "5V"
- board text added: "DIN"
- board text added: "DOUT"
- board text added: "GND"

Commit message: ordered
Added other boards and ordered all three
Connections:
- J1 pad 1: +5V -> Net-(D1-DIN)
- J1 pad 2: Net-(D1-DIN) -> +5V
- J2 pad 1: +5V -> Net-(D7-DOUT)
- J2 pad 2: Net-(D7-DOUT) -> +5V
Routing:
- net Net-(D1-DIN): track 27.9 -> 31.3 mm
- net Net-(D7-DOUT): track 8.38 -> 9.42 mm
Changed lines of the file:
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@@
 			(drillshape 0)
 			(scaleselection 1)
-			(outputdirectory "build/2026-08-08/")
+			(outputdirectory "build/2026-08-09")
 		)
 	)
@@
 			(remove_unused_layers no)
 			(roundrect_rratio 0.147059)
-			(net "+5V")
+			(net "Net-(D7-DOUT)")
 			(pinfunction "Pin_1_1")
 			(pintype "passive")
@@
 			(layers "*.Cu" "*.Mask")
 			(remove_unused_layers no)
-			(net "Net-(D7-DOUT)")
+			(net "+5V")
 			(pinfunction "Pin_2_2")
 			(pintype "passive")
@@
 			(remove_unused_layers no)
 			(roundrect_rratio 0.147059)
-			(net "+5V")
+			(net "Net-(D1-DIN)")
 			(pinfunction "Pin_1_1")
 			(pintype "passive")
@@
 			(layers "*.Cu" "*.Mask")
 			(remove_unused_layers no)
-			(net "Net-(D1-DIN)")
+			(net "+5V")
 			(pinfunction "Pin_2_2")
 			(pintype "passive")
@@
 		(end 90.319131 97.480832)
 		(stroke
-			(width 0)
+			(width 0.1)
 			(type default)
 		)
@@
 		(end 94.561772 101.723473)
 		(stroke
-			(width 0)
+			(width 0.1)
 			(type default)
 		)
@@
 		(end 90.319131 54.24264)
 		(stroke
-			(width 0)
+			(width 0.1)
 			(type default)
 		)
@@
 		(end 116.438227 101.723473)
 		(stroke
-			(width 0)
+			(width 0.1)
 			(type default)
 		)
@@
 		(end 107 64.680868)
 		(stroke
-			(width 0)
+			(width 0.1)
 			(type default)
 		)
@@
 		(end 107 87.042605)
 		(stroke
-			(width 0)
+			(width 0.1)
 			(type default)
 		)
@@
 		(end 94.561772 50)
 		(stroke
-			(width 0)
+			(width 0.1)
 			(type default)
 		)
@@
 		(end 120.680868 97.480832)
 		(stroke
-			(width 0)
-			(type default)
-		)
-		(layer "Dwgs.User")
-	)
-	(gr_line
-		(start 116.438227 101.723473)
-		(end 120.680868 97.480832)
-		(stroke
 			(width 0.1)
 			(type default)
 		)
-		(locked yes)
 		(layer "Dwgs.User")
 	)
@@
 		(end 116.438227 50)
 		(stroke
-			(width 0)
+			(width 0.1)
 			(type default)
 		)
@@
 		(end 120.680868 54.24264)
 		(stroke
-			(width 0)
+			(width 0.1)
 			(type default)
 		)
@@
 	)
 	(segment
-		(start 103.166652 54.395325)
-		(end 102.266652 53.495325)
+		(start 116.72052 67.898934)
+		(end 120.082375 71.260789)
 		(width 0.2)
 		(layer "F.Cu")
-		(net "Net-(D1-DIN)")
+		(net "Net-(D2-DOUT)")
 	)
 	(segment
-		(start 96.098529 76)
-		(end 103.166652 68.931877)
+		(start 120.082375 80.408396)
+		(end 116.690869 83.799902)
 		(width 0.2)
 		(layer "F.Cu")
-		(net "Net-(D1-DIN)")
+		(net "Net-(D2-DOUT)")
 	)
 	(segment
-		(start 103.166652 68.931877)
-		(end 103.166652 54.395325)
+		(start 120.082375 71.260789)
+		(end 120.082375 80.408396)
 		(width 0.2)
 		(layer "F.Cu")
-		(net "Net-(D1-DIN)")
-	)
-	(segment
-		(start 94 76)
-		(end 96.098529 76)
-		(width 0.2)
-		(layer "F.Cu")
-		(net "Net-(D1-DIN)")
+		(net "Net-(D2-DOUT)")
 	)
 	(segment
@@
 	)
 	(segment
-		(start 116.72052 67.898934)
-		(end 120.082375 71.260789)
+		(start 102.22987 98.215913)
+		(end 94.317575 90.303618)
 		(width 0.2)
 		(layer "F.Cu")
-		(net "Net-(D2-DOUT)")
+		(net "Net-(D4-DOUT)")
 	)
 	(segment
-		(start 120.082375 80.408396)
-		(end 116.690869 83.799902)
+		(start 102.253108 98.215913)
+		(end 102.22987 98.215913)
 		(width 0.2)
 		(layer "F.Cu")
-		(net "Net-(D2-DOUT)")
-	)
-	(segment
-		(start 120.082375 71.260789)
-		(end 120.082375 80.408396)
-		(width 0.2)
-		(layer "F.Cu")
-		(net "Net-(D2-DOUT)")
+		(net "Net-(D4-DOUT)")
 	)
 	(segment
@@
 		(layer "F.Cu")
 		(net "Net-(D3-DOUT)")
-	)
-	(segment
-		(start 102.22987 98.215913)
-		(end 94.317575 90.303618)
-		(width 0.2)
-		(layer "F.Cu")
-		(net "Net-(D4-DOUT)")
-	)
-	(segment
-		(start 102.253108 98.215913)
-		(end 102.22987 98.215913)
-		(width 0.2)
-		(layer "F.Cu")
-		(net "Net-(D4-DOUT)")
 	)
 	(segment
@@
 	)
 	(segment
+		(start 117 73)
+		(end 111.616759 73)
+		(width 0.2)
+		(layer "F.Cu")
+		(net "Net-(D7-DOUT)")
+	)
+	(segment
+		(start 111.616759 73)
+		(end 108.762521 75.854238)
+		(width 0.2)
+		(layer "F.Cu")
+		(net "Net-(D7-DOUT)")
+	)
+	(segment
 		(start 94.684217 61.434217)
 		(end 102.25 69)
@@
 	)
 	(segment
-		(start 108.762521 75.854238)
-		(end 116.645762 75.854238)
+		(start 104.25 70.25)
+		(end 104.25 68)
 		(width 0.2)
 		(layer "F.Cu")
-		(net "Net-(D7-DOUT)")
+		(net "Net-(D1-DIN)")
 	)
 	(segment
-		(start 116.645762 75.854238)
-		(end 117 75.5)
+		(start 102.266652 61.733348)
+		(end 102.266652 53.495325)
 		(width 0.2)
 		(layer "F.Cu")
-		(net "Net-(D7-DOUT)")
+		(net "Net-(D1-DIN)")
+	)
+	(segment
+		(start 94 78.5)
+		(end 96 78.5)
+		(width 0.2)
+		(layer "F.Cu")
+		(net "Net-(D1-DIN)")
+	)
+	(segment
+		(start 102.25 66)
+		(end 102.25 61.75)
+		(width 0.2)
+		(layer "F.Cu")
+		(net "Net-(D1-DIN)")
+	)
+	(segment
+		(start 96 78.5)
+		(end 104.25 70.25)
+		(width 0.2)
+		(layer "F.Cu")
+		(net "Net-(D1-DIN)")
+	)
+	(segment
+		(start 102.25 61.75)
+		(end 102.266652 61.733348)
+		(width 0.2)
+		(layer "F.Cu")
+		(net "Net-(D1-DIN)")
+	)
+	(segment
+		(start 104.25 68)
+		(end 102.25 66)
+		(width 0.2)
+		(layer "F.Cu")
+		(net "Net-(D1-DIN)")
 	)
 	(zone
